Commit message: [TEMP]: another temp update

File: workspace/src/slam_robots/robot/camera.xacro (robot description, xacro)
@@ -59,4 +59,5 @@
             <!-- actual plugin takes reads from transformed image even the sensor is attached to the 'camera_link', we want 'camera_link_optical' -->
             <plugin name="camera_controller" filename="libgazebo_ros_camera.so">
+                <xacro:if value="$(arg robot1)"><namespace>/robot1</namespace></xacro:if>
                 <frame_name>camera_link_optical</frame_name>
             </plugin>

File: workspace/src/slam_robots/robot/depth_camera.xacro (robot description, xacro)
@@ -41,4 +41,7 @@
             <plugin name="camera_controller" filename="libgazebo_ros_camera.so">
                 <frame_name>camera_link_optical</frame_name>
+                <!-- <ros> -->
+                    <!-- <xacro:if value="$(arg robot1)"><namespace>/robot1</namespace></xacro:if> -->
+                <!-- </ros> -->
                 <!-- still don't know the use of these depth as far and near are defined -->
                 <min_depth>0.1</min_depth>

File: workspace/src/slam_robots/robot/gazebo_control.xacro (robot description, xacro)
@@ -1,7 +1,13 @@
 <?xml version="1.0"?>
 <robot xmlns:xacro="http://www.ros.org/wiki/xacro">
+    <xacro:property name="suffix" value="$(arg number)"/>
     <gazebo>
         <!-- <plugin name="ignition::gazebo::systems::DiffDrive" filename="libignition-gazebo-diff-drive-system.so"> -->
         <plugin name='diff_drive' filename='libgazebo_ros_diff_drive.so'>
+            <!-- <ros> -->
+                <!-- <xacro:if value="$(arg robot1)"><namespace>/robot1</namespace></xacro:if> -->
+                <!-- <xacro:if value="$(arg robot2)"><namespace>/robot2</namespace></xacro:if> -->
+                <!-- <xacro:if value="$(arg robot3)"><namespace>/robot3</namespace></xacro:if> -->
+            <!-- </ros>  -->
             <!-- Wheel Information -->
             <left_joint>left_wheel_joint</left_joint>

File: workspace/src/slam_robots/robot/lidar.xacro (robot description, xacro)
@@ -71,4 +71,5 @@
                 <ros>
                     <argument>~/out:=scan</argument>
+                    <!-- <xacro:if value="$(arg robot1)"><namespace>/robot1</namespace></xacro:if> -->
                 </ros>
                 <!-- type of message output -->

File: workspace/src/slam_robots/robot/robot.urdf.xacro (robot description, xacro)
@@ -1,11 +1,13 @@
 <?xml version="1.0"?>
 <robot xmlns:xacro="http://www.ros.org/wiki/xacro"  name="robot">
+    <!-- xacro readme: https://github.com/ros/xacro/wiki#xacroinclude  -->
     <!-- <xacro:arg name="use_ros2_control" default="true"/> -->
-    <xacro:arg name="use_ros2_control" default="false"/>
-    <xacro:arg name="sim_mode" default="false"/>
+    <!-- <xacro:arg name="robot1" default="false"/> -->
+    <!-- <xacro:arg name="robot2" default="false"/> -->
+    <!-- <xacro:arg name="robot3" default="false"/> -->
     <!-- contains robot core shape -->
     <xacro:include filename="robot_core.xacro" />
     <!-- contains gazebo plugins-->
-    <xacro:include filename="gazebo_control.xacro" />
+    <xacro:include filename="gazebo_control.xacro" ns='other' />
     <!-- for lidar sensor -->
     <xacro:include filename="lidar.xacro" />
@@ -17,10 +19,3 @@
     <!-- add smily face to the robot -->
     <xacro:include filename="face.xacro" />
-    <!--  <xacro:if value="$(arg use_ros2_control)">
-        <xacro:include filename="ros2_control.xacro" />
-    </xacro:if>
-    <xacro:unless value="$(arg use_ros2_control)">
-        <xacro:include filename="gazebo_control.xacro" />
-    </xacro:unless>
-     -->
 </robot>
